Commit message: june 18

File: src/gazebo_example/models/xacro/example_robot.urdf.xacro (robot description, xacro)
@@ -4,5 +4,5 @@
   <xacro:macro name="plane_xacro" params="name:=robot">
     <gazebo>
-      <plugin filename="/home/silvos/Works/gazebo_ws/devel/lib/libgazebo_plane.so" name="gazebo_plane">
+      <plugin filename="/home/eitan/gazebo_example/devel/lib/libgazebo_plane.so" name="gazebo_plane">
         <robotNamespace>${name}</robotNamespace>
       </plugin>
@@ -10,7 +10,7 @@
     <link name="${name}_link">
       <inertial>
-        <mass value="1"/>
+        <mass value=".45"/>
         <origin xyz="0 0 0"/>
-        <inertia ixx="1" ixy="0.0" ixz="0.0" iyy="1" iyz="0.0" izz="1"/>
+        <inertia ixx="0.003922" ixy="0.0" ixz="0.0" iyy="0.01594" iyz="0.0" izz="0.01934"/>
       </inertial>
       <visual>
@@ -27,4 +27,199 @@
       </collision>
     </link>
+  <joint name="camera_joint" type="fixed">
+    <axis xyz="0 1 0" />
+    <origin xyz=".05 0 .9" rpy="0 0 0"/>
+    <parent link="${name}_link"/>
+    <child link="kinect"/>
+  </joint>
+  <!-- Camera -->
+  <link name="kinect">
+    <collision>
+      <origin xyz="0 0 0" rpy="0 0 0"/>
+      <geometry>
+    <box size="0.073000 0.276000 0.072000"/>
+      </geometry>
+    </collision>
+    <visual>
+      <origin xyz="0 0 0" rpy="0 0 0"/>
+      <geometry>
+    <box size="0.073000 0.276000 0.072000"/>
+      </geometry>
+      <material name="red"/>
+    </visual>
+    <inertial>
+      <mass value="1e-5" />
+      <origin xyz="0 0 0" rpy="0 0 0"/>
+      <inertia ixx="1e-6" ixy="0" ixz="0" iyy="1e-6" iyz="0" izz="1e-6" />
+    </inertial>
+  </link>
+    <gazebo reference="kinect">
+    <sensor type="depth" name="camera">
+      <update_rate>20.0</update_rate>
+      <camera>
+        <horizontal_fov>1.047198</horizontal_fov>
+        <image>
+          <width>640</width>
+          <height>480</height>
+          <format>R8G8B8</format>
+        </image>
+        <clip>
+          <near>0.05</near>
+          <far>3</far>
+        </clip>
+      </camera>
+        <plugin name="camera_plugin" filename="libgazebo_ros_openni_kinect.so">
+          <baseline>0.2</baseline>
+          <alwaysOn>true</alwaysOn>
+          <updateRate>0.0</updateRate>
+          <cameraName>camera_ir</cameraName>
+          <imageTopicName>/camera/depth/image_raw</imageTopicName>
+          <cameraInfoTopicName>/camera/depth/camera_info</cameraInfoTopicName>
+          <depthImageTopicName>/camera/depth/image_raw</depthImageTopicName>
+          <depthImageInfoTopicName>/camera/depth/camera_info</depthImageInfoTopicName>
+          <pointCloudTopicName>/camera/depth/points</pointCloudTopicName>
+          <frameName>camera_link</frameName>
+          <pointCloudCutoff>0.05</pointCloudCutoff>
+          <distortionK1>0</distortionK1>
+          <distortionK2>0</distortionK2>
+          <distortionK3>0</distortionK3>
+          <distortionT1>0</distortionT1>
+          <distortionT2>0</distortionT2>
+          <CxPrime>0</CxPrime>
+          <Cx>0</Cx>
+          <Cy>0</Cy>
+          <focalLength>0</focalLength>
+          <hackBaseline>0</hackBaseline>
+        </plugin>
+    </sensor>
+  </gazebo>
+  <!--<joint name="camera_joint" type="fixed">
+    <axis xyz="0 1 0" />
+    <origin xyz=".05 0 .9" rpy="0 0 0"/>
+    <parent link="${name}_link"/>
+    <child link="camera_link"/>
+  </joint>
+  <link name="camera_link">
+    <collision>
+      <origin xyz="0 0 0" rpy="0 0 0"/>
+      <geometry>
+    <box size=".05 .05 .05"/>
+      </geometry>
+    </collision>
+    <visual>
+      <origin xyz="0 0 0" rpy="0 0 0"/>
+      <geometry>
+    <box size=".05 .05 .05"/>
+      </geometry>
+      <material name="red"/>
+    </visual>
+    <inertial>
+      <mass value="1e-5" />
+      <origin xyz="0 0 0" rpy="0 0 0"/>
+      <inertia ixx="1e-6" ixy="0" ixz="0" iyy="1e-6" iyz="0" izz="1e-6" />
+    </inertial>
+  </link>-->
+  <!-- camera -->
+  <gazebo reference="camera_link1">
+    <sensor type="camera" name="camera1">
+      <update_rate>30.0</update_rate>
+      <camera name="head">
+        <horizontal_fov>1.3962634</horizontal_fov>
+        <image>
+          <width>800</width>
+          <height>800</height>
+          <format>R8G8B8</format>
+        </image>
+        <clip>
+          <near>0.02</near>
+          <far>300</far>
+        </clip>
+        <noise>
+          <type>gaussian</type>
+          <!-- Noise is sampled independently per pixel on each frame.
+               That pixel's noise value is added to each of its color
+               channels, which at that point lie in the range [0,1]. -->
+          <mean>0.0</mean>
+          <stddev>0.007</stddev>
+        </noise>
+      </camera>
+      <plugin name="camera_controller" filename="libgazebo_ros_camera.so">
+        <alwaysOn>true</alwaysOn>
+        <updateRate>0.0</updateRate>
+        <cameraName>rrbot/camera1</cameraName>
+        <imageTopicName>image_raw</imageTopicName>
+        <cameraInfoTopicName>camera_info</cameraInfoTopicName>-->
+        <frameName>camera_link_optical</frameName>
+        <!-- setting hackBaseline to anything but 0.0 will cause a misalignment
+            between the gazebo sensor image and the frame it is supposed to
+            be attached to -->
+        <hackBaseline>0.0</hackBaseline>
+        <distortionK1>0.0</distortionK1>
+        <distortionK2>0.0</distortionK2>
+        <distortionK3>0.0</distortionK3>
+        <distortionT1>0.0</distortionT1>
+        <distortionT2>0.0</distortionT2>
+        <CxPrime>0</CxPrime>
+        <Cx>0.0</Cx>
+        <Cy>0.0</Cy>
+        <focalLength>0.0</focalLength>
+      </plugin>
+    </sensor>
+  </gazebo>
+    <gazebo reference="camera_link2">
+    <sensor type="multicamera" name="stereo_camera">
+      <update_rate>30.0</update_rate>
+      <camera name="left">
+        <horizontal_fov>1.3962634</horizontal_fov>
+        <image>
+          <width>800</width>
+          <height>800</height>
+          <format>R8G8B8</format>
+        </image>
+        <clip>
+          <near>0.02</near>
+          <far>300</far>
+        </clip>
+        <noise>
+          <type>gaussian</type>
+          <mean>0.0</mean>
+          <stddev>0.007</stddev>
+        </noise>
+      </camera>
+      <camera name="right">
+        <pose>0 -0.07 0 0 0 0</pose>
+        <horizontal_fov>1.3962634</horizontal_fov>
+        <image>
+          <width>800</width>
+          <height>800</height>
+          <format>R8G8B8</format>
+        </image>
+        <clip>
+          <near>0.02</near>
+          <far>300</far>
+        </clip>
+        <noise>
+          <type>gaussian</type>
+          <mean>0.0</mean>
+          <stddev>0.007</stddev>
+        </noise>
+      </camera>
+      <plugin name="stereo_camera_controller" filename="libgazebo_ros_multicamera.so">
+        <alwaysOn>true</alwaysOn>
+        <updateRate>0.0</updateRate>
+        <cameraName>multisense_sl/camera</cameraName>
+        <imageTopicName>image_raw</imageTopicName>
+        <cameraInfoTopicName>camera_info</cameraInfoTopicName>
+        <frameName>left_camera_optical_frame</frameName>
+        <!--<rightFrameName>right_camera_optical_frame</rightFrameName>-->
+        <hackBaseline>0.07</hackBaseline>
+        <distortionK1>0.0</distortionK1>
+        <distortionK2>0.0</distortionK2>
+        <distortionK3>0.0</distortionK3>
+        <distortionT1>0.0</distortionT1>
+        <distortionT2>0.0</distortionT2>
+      </plugin>
+    </sensor>
+  </gazebo>
   </xacro:macro>
   <xacro:plane_xacro name="$(arg robot_name)" />

Commit message: motion plan node update

File: src/gazebo_example/models/xacro/example_robot.urdf.xacro (robot description, xacro)
@@ -29,5 +29,5 @@
   <joint name="camera_joint" type="fixed">
     <axis xyz="0 1 0" />
-    <origin xyz=".05 0 .9" rpy="0 0 0"/>
+    <origin xyz=".2 0 .2" rpy="0 0 0"/>
     <parent link="${name}_link"/>
     <child link="kinect"/>
@@ -49,7 +49,7 @@
     </visual>
     <inertial>
-      <mass value="1e-5" />
-      <origin xyz="0 0 0" rpy="0 0 0"/>
-      <inertia ixx="1e-6" ixy="0" ixz="0" iyy="1e-6" iyz="0" izz="1e-6" />
+      <mass value="1e-19" />
+      <origin xyz="0 0 0" rpy="0 0 0"/>
+      <inertia ixx="1e-19" ixy="0" ixz="0" iyy="1e-19" iyz="0" izz="1e-19" />
     </inertial>
   </link>
@@ -66,5 +66,5 @@
         <clip>
           <near>0.05</near>
-          <far>3</far>
+          <far>10</far>
         </clip>
       </camera>
@@ -78,5 +78,5 @@
           <depthImageTopicName>/camera/depth/image_raw</depthImageTopicName>
           <depthImageInfoTopicName>/camera/depth/camera_info</depthImageInfoTopicName>
-          <pointCloudTopicName>/camera/depth/points</pointCloudTopicName>
+          <pointCloudTopicName>/plane_xacro_default/points</pointCloudTopicName>
           <frameName>camera_link</frameName>
           <pointCloudCutoff>0.05</pointCloudCutoff>

Commit message: working trajectory distance check

File: src/gazebo_example/models/xacro/example_robot.urdf.xacro (robot description, xacro)
@@ -23,5 +23,5 @@
         <origin rpy="0 0 0" xyz="0 0 0"/>
         <geometry>
-          <mesh filename="package://gazebo_example/meshes/plane.dae"/>
+          <box size="0.2 1.0 0.2"/>
         </geometry>
       </collision>
@@ -56,14 +56,14 @@
     <gazebo reference="kinect">
     <sensor type="depth" name="camera">
-      <update_rate>20.0</update_rate>
+      <update_rate>90.0</update_rate>
       <camera>
-        <horizontal_fov>1.047198</horizontal_fov>
+        <horizontal_fov>1.50098</horizontal_fov>
         <image>
-          <width>640</width>
-          <height>480</height>
+          <width>1280</width>
+          <height>720</height>
           <format>R8G8B8</format>
         </image>
         <clip>
-          <near>0.05</near>
+          <near>0.2</near>
           <far>10</far>
         </clip>
@@ -94,132 +94,4 @@
     </sensor>
   </gazebo>
-  <!--<joint name="camera_joint" type="fixed">
-    <axis xyz="0 1 0" />
-    <origin xyz=".05 0 .9" rpy="0 0 0"/>
-    <parent link="${name}_link"/>
-    <child link="camera_link"/>
-  </joint>
-  <link name="camera_link">
-    <collision>
-      <origin xyz="0 0 0" rpy="0 0 0"/>
-      <geometry>
-    <box size=".05 .05 .05"/>
-      </geometry>
-    </collision>
-    <visual>
-      <origin xyz="0 0 0" rpy="0 0 0"/>
-      <geometry>
-    <box size=".05 .05 .05"/>
-      </geometry>
-      <material name="red"/>
-    </visual>
-    <inertial>
-      <mass value="1e-5" />
-      <origin xyz="0 0 0" rpy="0 0 0"/>
-      <inertia ixx="1e-6" ixy="0" ixz="0" iyy="1e-6" iyz="0" izz="1e-6" />
-    </inertial>
-  </link>-->
-  <!-- camera -->
-  <gazebo reference="camera_link1">
-    <sensor type="camera" name="camera1">
-      <update_rate>30.0</update_rate>
-      <camera name="head">
-        <horizontal_fov>1.3962634</horizontal_fov>
-        <image>
-          <width>800</width>
-          <height>800</height>
-          <format>R8G8B8</format>
-        </image>
-        <clip>
-          <near>0.02</near>
-          <far>300</far>
-        </clip>
-        <noise>
-          <type>gaussian</type>
-          <!-- Noise is sampled independently per pixel on each frame.
-               That pixel's noise value is added to each of its color
-               channels, which at that point lie in the range [0,1]. -->
-          <mean>0.0</mean>
-          <stddev>0.007</stddev>
-        </noise>
-      </camera>
-      <plugin name="camera_controller" filename="libgazebo_ros_camera.so">
-        <alwaysOn>true</alwaysOn>
-        <updateRate>0.0</updateRate>
-        <cameraName>rrbot/camera1</cameraName>
-        <imageTopicName>image_raw</imageTopicName>
-        <cameraInfoTopicName>camera_info</cameraInfoTopicName>-->
-        <frameName>camera_link_optical</frameName>
-        <!-- setting hackBaseline to anything but 0.0 will cause a misalignment
-            between the gazebo sensor image and the frame it is supposed to
-            be attached to -->
-        <hackBaseline>0.0</hackBaseline>
-        <distortionK1>0.0</distortionK1>
-        <distortionK2>0.0</distortionK2>
-        <distortionK3>0.0</distortionK3>
-        <distortionT1>0.0</distortionT1>
-        <distortionT2>0.0</distortionT2>
-        <CxPrime>0</CxPrime>
-        <Cx>0.0</Cx>
-        <Cy>0.0</Cy>
-        <focalLength>0.0</focalLength>
-      </plugin>
-    </sensor>
-  </gazebo>
-    <gazebo reference="camera_link2">
-    <sensor type="multicamera" name="stereo_camera">
-      <update_rate>30.0</update_rate>
-      <camera name="left">
-        <horizontal_fov>1.3962634</horizontal_fov>
-        <image>
-          <width>800</width>
-          <height>800</height>
-          <format>R8G8B8</format>
-        </image>
-        <clip>
-          <near>0.02</near>
-          <far>300</far>
-        </clip>
-        <noise>
-          <type>gaussian</type>
-          <mean>0.0</mean>
-          <stddev>0.007</stddev>
-        </noise>
-      </camera>
-      <camera name="right">
-        <pose>0 -0.07 0 0 0 0</pose>
-        <horizontal_fov>1.3962634</horizontal_fov>
-        <image>
-          <width>800</width>
-          <height>800</height>
-          <format>R8G8B8</format>
-        </image>
-        <clip>
-          <near>0.02</near>
-          <far>300</far>
-        </clip>
-        <noise>
-          <type>gaussian</type>
-          <mean>0.0</mean>
-          <stddev>0.007</stddev>
-        </noise>
-      </camera>
-      <plugin name="stereo_camera_controller" filename="libgazebo_ros_multicamera.so">
-        <alwaysOn>true</alwaysOn>
-        <updateRate>0.0</updateRate>
-        <cameraName>multisense_sl/camera</cameraName>
-        <imageTopicName>image_raw</imageTopicName>
-        <cameraInfoTopicName>camera_info</cameraInfoTopicName>
-        <frameName>left_camera_optical_frame</frameName>
-        <!--<rightFrameName>right_camera_optical_frame</rightFrameName>-->
-        <hackBaseline>0.07</hackBaseline>
-        <distortionK1>0.0</distortionK1>
-        <distortionK2>0.0</distortionK2>
-        <distortionK3>0.0</distortionK3>
-        <distortionT1>0.0</distortionT1>
-        <distortionT2>0.0</distortionT2>
-      </plugin>
-    </sensor>
-  </gazebo>
   </xacro:macro>
   <xacro:plane_xacro name="$(arg robot_name)" />

Commit message: working rviz and obstacle avoidance is decent

File: src/gazebo_example/models/xacro/example_robot.urdf.xacro (robot description, xacro)
@@ -1,12 +1,14 @@
 <?xml version="1.0" ?>
-<robot name="example_robot_xacro" xmlns:xacro="http://www.ros.org/wiki/xacro">
-  <xacro:arg name="robot_name" default="plane_xacro_default"/>
-  <xacro:macro name="plane_xacro" params="name:=robot">
+<robot name="mcfoamy" xmlns:xacro="http://www.ros.org/wiki/xacro">
     <gazebo>
       <plugin filename="/home/eitan/mcfoamy_gazebo/devel/lib/libgazebo_plane.so" name="gazebo_plane">
-        <robotNamespace>${name}</robotNamespace>
-      </plugin>
+     </plugin>
     </gazebo>
-    <link name="${name}_link">
+    <link name="world"/>
+    <joint name="fixed" type="floating">
+      <parent link="world"/>
+      <child link="airframe"/>
+    </joint>
+    <link name="airframe">
       <inertial>
         <mass value=".45"/>
@@ -30,5 +32,5 @@
     <axis xyz="0 1 0" />
     <origin xyz=".2 0 .2" rpy="0 0 0"/>
-    <parent link="${name}_link"/>
+    <parent link="airframe"/>
     <child link="kinect"/>
   </joint>
@@ -78,6 +80,6 @@
           <depthImageTopicName>/camera/depth/image_raw</depthImageTopicName>
           <depthImageInfoTopicName>/camera/depth/camera_info</depthImageInfoTopicName>
-          <pointCloudTopicName>/plane_xacro_default/points</pointCloudTopicName>
-          <frameName>camera_link</frameName>
+          <pointCloudTopicName>/camera/depth/points</pointCloudTopicName>
+          <frameName>kinect_camera_frame</frameName>
           <pointCloudCutoff>0.2</pointCloudCutoff>
           <pointCloudCutoffMax>10.0</pointCloudCutoffMax>
@@ -95,5 +97,3 @@
     </sensor>
   </gazebo>
-  </xacro:macro>
-  <xacro:plane_xacro name="$(arg robot_name)" />
 </robot>

Commit message: up to date with icuas19 initial submission

File: src/gazebo_example/models/xacro/example_robot.urdf.xacro (robot description, xacro)
@@ -14,5 +14,5 @@
         <mass value=".45"/>
         <origin xyz="0 0 0"/>
-        <inertia ixx="0.003922" ixy="0.0" ixz="0.0" iyy="0.01594" iyz="0.0" izz="0.01934"/>
+        <inertia ixx="0.003922" ixy="0.0" ixz="0.000303" iyy="0.01594" iyz="0.0" izz="0.01934"/>
       </inertial>
       <visual>

Commit message: mcfoamy cad inserted

File: src/gazebo_example/models/xacro/example_robot.urdf.xacro (robot description, xacro)
@@ -19,5 +19,5 @@
         <origin rpy="0 0 0" xyz="0 0 0"/>
         <geometry>
-          <mesh filename="package://gazebo_example/meshes/plane.dae"/>
+          <mesh filename="package://gazebo_example/meshes/mcfoamy_mod.STL"/>
         </geometry>
       </visual>
@@ -30,6 +30,6 @@
     </link>
   <joint name="camera_joint" type="fixed">
-    <axis xyz="0 1 0" />
-    <origin xyz=".2 0 .2" rpy="0 0 0"/>
+    <axis xyz="1 0 0" />
+    <origin xyz="0 0 .15" rpy="0 0 0"/>
     <parent link="airframe"/>
     <child link="kinect"/>
@@ -62,11 +62,11 @@
         <horizontal_fov>1.50098</horizontal_fov>
         <image>
-          <width>1280</width>
-          <height>720</height>
+          <width>640</width>
+          <height>480</height>
           <format>R8G8B8</format>
         </image>
         <clip>
           <near>0.2</near>
-          <far>15</far>
+          <far>25</far>
         </clip>
       </camera>
@@ -83,5 +83,5 @@
           <frameName>kinect_camera_frame</frameName>
           <pointCloudCutoff>0.2</pointCloudCutoff>
-          <pointCloudCutoffMax>15.0</pointCloudCutoffMax>
+          <pointCloudCutoffMax>25.0</pointCloudCutoffMax>
           <distortionK1>0</distortionK1>
           <distortionK2>0</distortionK2>

Commit message: fixed time since trajectry received

File: src/gazebo_example/models/xacro/example_robot.urdf.xacro (robot description, xacro)
@@ -12,7 +12,7 @@
     <link name="airframe">
       <inertial>
-        <mass value=".45"/>
+        <mass value=".6"/>
         <origin xyz="0 0 0"/>
-        <inertia ixx="0.003922" ixy="0.0" ixz="0.000303" iyy="0.01594" iyz="0.0" izz="0.01934"/>
+        <inertia ixx="0.005" ixy="0.0" ixz="0.0" iyy="0.021" iyz="0.0" izz="0.023"/>
       </inertial>
       <visual>

Commit message: updated with only position derivitive and integrator

File: src/gazebo_example/models/xacro/example_robot.urdf.xacro (robot description, xacro)
@@ -1,4 +1,7 @@
 <?xml version="1.0" ?>
 <robot name="mcfoamy" xmlns:xacro="http://www.ros.org/wiki/xacro">
+    <material name="white">
+    <color rgba="1 1 1 1"/>
+  </material>
     <gazebo>
       <plugin filename="/home/eitan/mcfoamy_gazebo/devel/lib/libgazebo_plane.so" name="gazebo_plane">
@@ -21,4 +24,5 @@
           <mesh filename="package://gazebo_example/meshes/mcfoamy_mod.STL"/>
         </geometry>
+      <material name="white"/>
       </visual>
       <collision>
@@ -48,5 +52,5 @@
     <box size="0.073000 0.276000 0.072000"/>
       </geometry>
-      <material name="red"/>
+      <material name="white"/>
     </visual>
     <inertial>
@@ -83,5 +87,5 @@
           <frameName>kinect_camera_frame</frameName>
           <pointCloudCutoff>0.2</pointCloudCutoff>
-          <pointCloudCutoffMax>25.0</pointCloudCutoffMax>
+          <pointCloudCutoffMax>20.0</pointCloudCutoffMax>
           <distortionK1>0</distortionK1>
           <distortionK2>0</distortionK2>

Commit message: updated trajectories and aircraft properties and high velocity trajectory fix

File: src/gazebo_example/models/xacro/example_robot.urdf.xacro (robot description, xacro)
@@ -15,5 +15,5 @@
     <link name="airframe">
       <inertial>
-        <mass value=".6"/>
+        <mass value=".66"/>
         <origin xyz="0 0 0"/>
         <inertia ixx="0.005" ixy="0.0" ixz="0.0" iyy="0.021" iyz="0.0" izz="0.023"/>
